File: eagle/BattLogg/main.sch (EAGLE design)
At the start: 5 parts, among them U1 ADAFRUIT_ADS1115, U2 ADAFRUIT_ADS1115, U3 ADAFRUIT_ADS1115, U4 ADAFRUIT_ADS1115

Commit message: init
Parts:
- added U$1: STM32F4V_100PIN_GPSBOARD, stm32f4:STM32F4V_100PIN_GPSBOARD
Connections:
- removed net N$4: U$2.VSS, U1.GND, U2.GND, U3.GND, U4.ADDR, U4.GND
- new net GND: U$1.VSS1, U$1.VSS2, U$1.VSS3, U$2.VSS, U1.GND, U2.GND, U3.GND, U4.ADDR, U4.GND
- net N$1: now also U$1.PB7
- net N$3: now also U$1.PB6
Changed lines of the file:
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@@
 <layer number="2" name="Route2" color="1" fill="3" visible="no" active="no"/>
 <layer number="3" name="Route3" color="4" fill="3" visible="no" active="no"/>
+<layer number="4" name="Route4" color="1" fill="4" visible="no" active="no"/>
+<layer number="5" name="Route5" color="4" fill="4" visible="no" active="no"/>
+<layer number="6" name="Route6" color="1" fill="8" visible="no" active="no"/>
+<layer number="7" name="Route7" color="4" fill="8" visible="no" active="no"/>
+<layer number="8" name="Route8" color="1" fill="2" visible="no" active="no"/>
+<layer number="9" name="Route9" color="4" fill="2" visible="no" active="no"/>
+<layer number="10" name="Route10" color="1" fill="7" visible="no" active="no"/>
+<layer number="11" name="Route11" color="4" fill="7" visible="no" active="no"/>
+<layer number="12" name="Route12" color="1" fill="5" visible="no" active="no"/>
+<layer number="13" name="Route13" color="4" fill="5" visible="no" active="no"/>
 <layer number="14" name="Route14" color="1" fill="6" visible="no" active="no"/>
 <layer number="15" name="Route15" color="4" fill="6" visible="no" active="no"/>
@@
 <part name="U3" library="AD convertor" deviceset="ADAFRUIT_ADS1115" device=""/>
 <part name="U4" library="AD convertor" deviceset="ADAFRUIT_ADS1115" device=""/>
+<part name="U$1" library="stm32f4" deviceset="STM32F4V_100PIN_GPSBOARD" device=""/>
+<part name="GND1" library="supply1" library_urn="urn:adsk.eagle:library:371" deviceset="GND" device=""/>
+<part name="GND2" library="supply1" library_urn="urn:adsk.eagle:library:371" deviceset="GND" device=""/>
 </parts>
 <sheets>
@@
 <attribute name="VALUE" x="134.62" y="167.64" size="1.27" layer="95"/>
 </instance>
+<instance part="U$1" gate="G$1" x="22.86" y="152.4" smashed="yes"/>
+<instance part="GND1" gate="1" x="17.78" y="58.42" smashed="yes">
+<attribute name="VALUE" x="15.24" y="55.88" size="1.778" layer="96"/>
+</instance>
+<instance part="GND2" gate="1" x="157.48" y="66.04" smashed="yes">
+<attribute name="VALUE" x="154.94" y="63.5" size="1.778" layer="96"/>
+</instance>
 </instances>
 <busses>
@@
 <net name="N$1" class="0">
 <segment>
-<wire x1="77.47" y1="113.03" x2="109.22" y2="113.03" width="0.1524" layer="91"/>
 <pinref part="U1" gate="G$1" pin="SDA"/>
-<wire x1="109.22" y1="113.03" x2="109.22" y2="106.68" width="0.1524" layer="91"/>
 <wire x1="109.22" y1="106.68" x2="127" y2="106.68" width="0.1524" layer="91"/>
 <pinref part="U2" gate="G$1" pin="SDA"/>
-<wire x1="109.22" y1="113.03" x2="109.22" y2="132.08" width="0.1524" layer="91"/>
+<wire x1="109.22" y1="106.68" x2="109.22" y2="132.08" width="0.1524" layer="91"/>
 <wire x1="109.22" y1="132.08" x2="124.46" y2="132.08" width="0.1524" layer="91"/>
 <pinref part="U3" gate="G$1" pin="SDA"/>
@@
 <wire x1="124.46" y1="129.54" x2="124.46" y2="132.08" width="0.1524" layer="91"/>
 <junction x="124.46" y="132.08"/>
+<pinref part="U$1" gate="G$1" pin="PB7"/>
+<wire x1="67.31" y1="191.77" x2="109.22" y2="191.77" width="0.1524" layer="91"/>
+<wire x1="109.22" y1="191.77" x2="109.22" y2="182.88" width="0.1524" layer="91"/>
+<junction x="109.22" y="182.88"/>
 </segment>
 </net>
@@
 <wire x1="127" y1="134.62" x2="111.76" y2="134.62" width="0.1524" layer="91"/>
 <wire x1="111.76" y1="134.62" x2="111.76" y2="109.22" width="0.1524" layer="91"/>
-<wire x1="77.47" y1="110.49" x2="77.47" y2="109.22" width="0.1524" layer="91"/>
-<wire x1="77.47" y1="109.22" x2="111.76" y2="109.22" width="0.1524" layer="91"/>
 <pinref part="U1" gate="G$1" pin="SCL"/>
 <wire x1="111.76" y1="109.22" x2="121.92" y2="109.22" width="0.1524" layer="91"/>
-<junction x="111.76" y="109.22"/>
 <pinref part="U3" gate="G$1" pin="SCL"/>
 <wire x1="121.92" y1="109.22" x2="127" y2="109.22" width="0.1524" layer="91"/>
@@
 <wire x1="121.92" y1="104.14" x2="121.92" y2="109.22" width="0.1524" layer="91"/>
 <junction x="121.92" y="109.22"/>
+<pinref part="U$1" gate="G$1" pin="PB6"/>
+<wire x1="111.76" y1="185.42" x2="111.76" y2="189.23" width="0.1524" layer="91"/>
+<wire x1="111.76" y1="189.23" x2="67.31" y2="189.23" width="0.1524" layer="91"/>
+<junction x="111.76" y="185.42"/>
 </segment>
 </net>
@@
 </segment>
 </net>
-<net name="N$4" class="0">
+<net name="GND" class="0">
 <segment>
 <pinref part="U4" gate="G$1" pin="GND"/>
@@
 <wire x1="127" y1="111.76" x2="116.84" y2="111.76" width="0.1524" layer="91"/>
 <junction x="116.84" y="111.76"/>
+<pinref part="GND2" gate="1" pin="GND"/>
+<wire x1="157.48" y1="68.58" x2="157.48" y2="71.12" width="0.1524" layer="91"/>
+<wire x1="157.48" y1="71.12" x2="154.94" y2="71.12" width="0.1524" layer="91"/>
+<junction x="154.94" y="71.12"/>
+</segment>
+<segment>
+<pinref part="GND1" gate="1" pin="GND"/>
+<pinref part="U$1" gate="G$1" pin="VSS2"/>
+<wire x1="17.78" y1="60.96" x2="17.78" y2="63.5" width="0.1524" layer="91"/>
+<pinref part="U$1" gate="G$1" pin="VSS3"/>
+<wire x1="20.32" y1="63.5" x2="17.78" y2="63.5" width="0.1524" layer="91"/>
+<junction x="17.78" y="63.5"/>
+<pinref part="U$1" gate="G$1" pin="VSS1"/>
+<wire x1="17.78" y1="63.5" x2="15.24" y2="63.5" width="0.1524" layer="91"/>
 </segment>
 </net>
@@
 </schematic>
 </drawing>
+<compatibility>
+<note version="8.2" severity="warning">
+Since Version 8.2, EAGLE supports online libraries. The ids
+of those online libraries will not be understood (or retained)
+with this version.
+</note>
+<note version="8.3" severity="warning">
+Since Version 8.3, EAGLE supports URNs for individual library
+assets (packages, symbols, and devices). The URNs of those assets
+will not be understood (or retained) with this version.
+</note>
+</compatibility>
 </eagle>
